Commit message: Added camera module to AgileX

File: src/agilex_scout/agilex_scout_description/urdf/robot/scout_v2.urdf.xacro (robot description, xacro)
@@ -93,4 +93,48 @@
 			<xacro:include filename="$(find agilex_scout_description)/urdf/robot/scout_v2.gazebo" />
 		</xacro:if>
+		<!-- Camera: ADDED TO HAVE IMAGES FOR THE MEMORY GRAPH -->
+		<link name="camera_link">
+            <visual>
+                <geometry>
+                    <box size="0.05 0.05 0.05"/>
+                </geometry>
+                <material name="black">
+                    <color rgba="0 0 0 1"/>
+                </material>
+            </visual>
+            <collision>
+                <geometry>
+                    <box size="0.05 0.05 0.05"/>
+                </geometry>
+            </collision>
+            <inertial>
+                <mass value="0.1"/>
+                <inertia ixx="0.0001" ixy="0" ixz="0" iyy="0.0001" iyz="0" izz="0.0001"/>
+            </inertial>
+        </link>
+        <joint name="camera_joint" type="fixed">
+            <origin xyz="0.05 0 0.05" rpy="0 0 0"/>
+            <parent link="front_mount"/>
+            <child link="camera_link"/>
+        </joint>
+        <gazebo reference="camera_link">
+            <sensor name="scout_camera" type="camera">
+                <pose>0 0 0 0 0 0</pose>
+                <visualize>true</visualize>
+                <update_rate>30</update_rate>
+                <topic>camera/image_raw</topic> <camera>
+                    <horizontal_fov>1.047</horizontal_fov>
+                    <image>
+                        <width>640</width>
+                        <height>480</height>
+                        <format>R8G8B8</format>
+                    </image>
+                    <clip>
+                        <near>0.1</near>
+                        <far>100</far>
+                    </clip>
+                </camera>
+            </sensor>
+        </gazebo>
 	</xacro:macro>
 </robot>

Commit message: Working Nav2 stack

File: src/agilex_scout/agilex_scout_description/urdf/robot/scout_v2.urdf.xacro (robot description, xacro)
@@ -93,48 +93,4 @@
 			<xacro:include filename="$(find agilex_scout_description)/urdf/robot/scout_v2.gazebo" />
 		</xacro:if>
-		<!-- Camera: ADDED TO HAVE IMAGES FOR THE MEMORY GRAPH -->
-		<link name="camera_link">
-            <visual>
-                <geometry>
-                    <box size="0.05 0.05 0.05"/>
-                </geometry>
-                <material name="black">
-                    <color rgba="0 0 0 1"/>
-                </material>
-            </visual>
-            <collision>
-                <geometry>
-                    <box size="0.05 0.05 0.05"/>
-                </geometry>
-            </collision>
-            <inertial>
-                <mass value="0.1"/>
-                <inertia ixx="0.0001" ixy="0" ixz="0" iyy="0.0001" iyz="0" izz="0.0001"/>
-            </inertial>
-        </link>
-        <joint name="camera_joint" type="fixed">
-            <origin xyz="0.05 0 0.05" rpy="0 0 0"/>
-            <parent link="front_mount"/>
-            <child link="camera_link"/>
-        </joint>
-        <gazebo reference="camera_link">
-            <sensor name="scout_camera" type="camera">
-                <pose>0 0 0 0 0 0</pose>
-                <visualize>true</visualize>
-                <update_rate>30</update_rate>
-                <topic>camera/image_raw</topic> <camera>
-                    <horizontal_fov>1.047</horizontal_fov>
-                    <image>
-                        <width>640</width>
-                        <height>480</height>
-                        <format>R8G8B8</format>
-                    </image>
-                    <clip>
-                        <near>0.1</near>
-                        <far>100</far>
-                    </clip>
-                </camera>
-            </sensor>
-        </gazebo>
 	</xacro:macro>
 </robot>

Commit message: Refined working NAV2 tool (struggling under simulation frequency)

File: src/agilex_scout/agilex_scout_description/urdf/robot/scout_v2.urdf.xacro (robot description, xacro)
@@ -93,4 +93,48 @@
 			<xacro:include filename="$(find agilex_scout_description)/urdf/robot/scout_v2.gazebo" />
 		</xacro:if>
+		<!-- Camera: ADDED TO HAVE IMAGES FOR THE MEMORY GRAPH -->
+		<link name="camera_link">
+            <visual>
+                <geometry>
+                    <box size="0.05 0.05 0.05"/>
+                </geometry>
+                <material name="black">
+                    <color rgba="0 0 0 1"/>
+                </material>
+            </visual>
+            <collision>
+                <geometry>
+                    <box size="0.05 0.05 0.05"/>
+                </geometry>
+            </collision>
+            <inertial>
+                <mass value="0.1"/>
+                <inertia ixx="0.0001" ixy="0" ixz="0" iyy="0.0001" iyz="0" izz="0.0001"/>
+            </inertial>
+        </link>
+        <joint name="camera_joint" type="fixed">
+            <origin xyz="0.05 0 0.05" rpy="0 0 0"/>
+            <parent link="front_mount"/>
+            <child link="camera_link"/>
+        </joint>
+        <gazebo reference="camera_link">
+            <sensor name="scout_camera" type="camera">
+                <pose>0 0 0 0 0 0</pose>
+                <visualize>true</visualize>
+                <update_rate>30</update_rate>
+                <topic>camera/image_raw</topic> <camera>
+                    <horizontal_fov>1.2</horizontal_fov>
+                    <image>
+                        <width>1920</width>
+                        <height>1080</height>
+                        <format>R8G8B8</format>
+                    </image>
+                    <clip>
+                        <near>0.1</near>
+                        <far>100</far>
+                    </clip>
+                </camera>
+            </sensor>
+        </gazebo>
 	</xacro:macro>
 </robot>
